File: Ethernet_Dev_Board/Ethernet_Dev_Board.kicad_sch (KiCad schematic)
At the start: 27 parts, among them J101 Power In, J102 5V, J103 3.3V, J104 3.3VA, J105 3.3VD, U101 AZ1117

Commit message: Generated PCB file from schematic
Parts:
- J106: footprint LED_Controller_Hardware:WIZNET_RB1-125BAG1A -> RG_Connectors:WIZNET_RB1-125BAG1A
Changed lines of the file:
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@@
 			)
 		)
-		(property "Footprint" "LED_Controller_Hardware:WIZNET_RB1-125BAG1A"
+		(property "Footprint" "RG_Connectors:WIZNET_RB1-125BAG1A"
 			(at 265.43 104.14 0)
 			(effects

Commit message: Associating footprint to component
Parts:
- J101: footprint LED_Controller_Hardware:CUI_TBP01R1-508-02BE -> RG_Terminals:CUI_TBP01R1-508-02BE
Changed lines of the file:
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@@
 			)
 		)
-		(property "Footprint" "LED_Controller_Hardware:CUI_TBP01R1-508-02BE"
+		(property "Footprint" "RG_Terminals:CUI_TBP01R1-508-02BE"
 			(at 50.165 86.36 0)
 			(effects
