File: Ethernet_Dev_Board/Ethernet_Dev_Board.kicad_sch (KiCad schematic)
At the start: 33 parts, among them J101 Power In, U101 AZ1117, U102 74AUP1T08GWH, U103 1.2V

Commit message: Updated part(s) due to out of stock
Parts:
- C106, C107, C108, C111, C112: Distributor PN 1276-1274-2-ND -> 490-10476-2-ND; Mfg. Samsung Electro-Mechanics -> Murata Electronics; Mfg. PN CL10A226MP8NUNE -> GRM188R61A226ME15D
Changed lines of the file:
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@@
 			)
 		)
-		(property "Mfg." "Samsung Electro-Mechanics"
+		(property "Mfg." "Murata Electronics"
 			(at 99.06 104.14 0)
 			(effects
@@
 			)
 		)
-		(property "Mfg. PN" "CL10A226MP8NUNE"
+		(property "Mfg. PN" "GRM188R61A226ME15D"
 			(at 99.06 104.14 0)
 			(effects
@@
 			)
 		)
-		(property "Distributor PN" "1276-1274-2-ND"
+		(property "Distributor PN" "490-10476-2-ND"
 			(at 99.06 104.14 0)
 			(effects
@@
 			)
 		)
-		(property "Mfg." "Samsung Electro-Mechanics"
+		(property "Mfg." "Murata Electronics"
 			(at 87.636 37.471 0)
 			(effects
@@
 			)
 		)
-		(property "Mfg. PN" "CL10A226MP8NUNE"
+		(property "Mfg. PN" "GRM188R61A226ME15D"
 			(at 87.636 37.471 0)
 			(effects
@@
 			)
 		)
-		(property "Distributor PN" "1276-1274-2-ND"
+		(property "Distributor PN" "490-10476-2-ND"
 			(at 87.636 37.471 0)
 			(effects
@@
 			)
 		)
-		(property "Mfg." "Samsung Electro-Mechanics"
+		(property "Mfg." "Murata Electronics"
 			(at 88.9 104.14 0)
 			(effects
@@
 			)
 		)
-		(property "Mfg. PN" "CL10A226MP8NUNE"
+		(property "Mfg. PN" "GRM188R61A226ME15D"
 			(at 88.9 104.14 0)
 			(effects
@@
 			)
 		)
-		(property "Distributor PN" "1276-1274-2-ND"
+		(property "Distributor PN" "490-10476-2-ND"
 			(at 88.9 104.14 0)
 			(effects
@@
 			)
 		)
-		(property "Mfg." "Samsung Electro-Mechanics"
+		(property "Mfg." "Murata Electronics"
 			(at 99.06 82.55 0)
 			(effects
@@
 			)
 		)
-		(property "Mfg. PN" "CL10A226MP8NUNE"
+		(property "Mfg. PN" "GRM188R61A226ME15D"
 			(at 99.06 82.55 0)
 			(effects
@@
 			)
 		)
-		(property "Distributor PN" "1276-1274-2-ND"
+		(property "Distributor PN" "490-10476-2-ND"
 			(at 99.06 82.55 0)
 			(effects
@@
 			)
 		)
-		(property "Mfg." "Samsung Electro-Mechanics"
+		(property "Mfg." "Murata Electronics"
 			(at 88.9 82.55 0)
 			(effects
@@
 			)
 		)
-		(property "Mfg. PN" "CL10A226MP8NUNE"
+		(property "Mfg. PN" "GRM188R61A226ME15D"
 			(at 88.9 82.55 0)
 			(effects
@@
 			)
 		)
-		(property "Distributor PN" "1276-1274-2-ND"
+		(property "Distributor PN" "490-10476-2-ND"
 			(at 88.9 82.55 0)
 			(effects
