File: Ethernet_Dev_Board/W5100S_Dev.kicad_sch (KiCad schematic)
At the start: 41 parts, among them U302 74AUP1T08GWH, Y301 25MHz

Commit message: Added TVS diode and redid the LED circuit on the ESP32
Parts:
- Y301: footprint (none) -> RG_Crystal:Crystal_SMD_4Pin_3.2x2.5mm
Changed lines of the file:
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@@
 			)
 		)
-		(property "Footprint" ""
+		(property "Footprint" "RG_Crystal:Crystal_SMD_4Pin_3.2x2.5mm"
 			(at 29.21 193.04 0)
 			(effects
