File: Ethernet_Dev_Board/ESP32.kicad_sch (KiCad schematic)
At the start: 22 parts, among them J401 TAG-CONNECT_NL_10-POS_LEGS, U402 ESP32-WROOM-32E, U403 74LVC1G11W6

Commit message: Updated part(s) due to out of stock
Parts:
- C403: Distributor PN 1276-1274-2-ND -> 490-10476-2-ND; Mfg. Samsung Electro-Mechanics -> Murata Electronics; Mfg. PN CL10A226MP8NUNE -> GRM188R61A226ME15D
Changed lines of the file:
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@@
 			)
 		)
-		(property "Mfg." "Samsung Electro-Mechanics"
+		(property "Mfg." "Murata Electronics"
 			(at 91.44 46.99 0)
 			(effects
@@
 			)
 		)
-		(property "Mfg. PN" "CL10A226MP8NUNE"
+		(property "Mfg. PN" "GRM188R61A226ME15D"
 			(at 91.44 46.99 0)
 			(effects
@@
 			)
 		)
-		(property "Distributor PN" "1276-1274-2-ND"
+		(property "Distributor PN" "490-10476-2-ND"
 			(at 91.44 46.99 0)
 			(effects
